File: PCB/RS232-multiport.sch (KiCad schematic (older format))
At the start: 17 parts, among them J1 DB9_Male_MountingHoles, J2 DB9_Male_MountingHoles, J3 DB9_Male_MountingHoles, J4 DB9_Male_MountingHoles, U1 MAX232, U2 MAX232

Commit message: v2
Parts:
- added D1, D2, D3, D4, D5, D6, D7, D8: LED, LED_SMD:LED_1206_3216Metric_Pad1.42x1.75mm_HandSolder, symbol Device:LED
- added R1, R2, R3, R4, R5, R6, R7, R8: 4.7k, Resistor_SMD:R_1206_3216Metric_Pad1.42x1.75mm_HandSolder, symbol Device:R_US
- C1, C10, C2, C3, C4, C5, C6, C7, C8, C9: footprint Capacitor_THT:C_Radial_D6.3mm_H7.0mm_P2.50mm -> Capacitor_SMD:C_1206_3216Metric_Pad1.42x1.75mm_HandSolder
Connections:
- net at U1.13 (R1IN): now also J1.2, R2.1; no longer J1.4
- net at J1.3, U1.14 (T1OUT): now also R1.1
- net -10V: now reaches C8.1, U1.6 (VS-)
- net -10V: now also C10.1, U2.6 (VS-), D1.1 (K), D2.1 (K), D3.1 (K), D4.1 (K), D5.1 (K), D6.1 (K), D7.1 (K), D8.1 (K)
- net at J2.3, U1.7 (T2OUT): now also R3.1
- net at U1.8 (R2IN): now also J2.2, R4.1; no longer J2.4
- net at J3.2: now also U2.13 (R1IN), R6.1
- net at J3.3, U2.14 (T1OUT): now also R5.1
- net at J3.4: no longer U2.13 (R1IN)
- net at J4.2: now also U2.8 (R2IN), R8.1
- net at J4.3, U2.7 (T2OUT): now also R7.1
- net at J4.4: no longer U2.8 (R2IN)
- new net: D1.2 (A), R1.2
- new net: D2.2 (A), R2.2
- new net: D3.2 (A), R3.2
- new net: D4.2 (A), R4.2
- new net: D5.2 (A), R5.2
- new net: D6.2 (A), R6.2
- new net: D7.2 (A), R7.2
- new net: D8.2 (A), R8.2
Other:
- moved on the sheet: C10, C8
